Commit message: fix: joint angle limit updated

File: rbpodo_description/robots/rb5_850e.urdf (robot description, URDF)
Before this commit: robot rb5_850e, 8 links, 7 joints
Joints:
- joint base: limit lower=-3.14 upper=3.14 effort=10 velocity=3.14 -> lower=-6.0 upper=6.0 effort=10 velocity=3.14
- joint shoulder: limit lower=-3.14 upper=3.14 effort=10 velocity=3.14 -> lower=-6.0 upper=6.0 effort=10 velocity=3.14
- joint wrist1: limit lower=-3.14 upper=3.14 effort=10 velocity=3.14 -> lower=-6.0 upper=6.0 effort=10 velocity=3.14
- joint wrist2: limit lower=-3.14 upper=3.14 effort=10 velocity=3.14 -> lower=-6.0 upper=6.0 effort=10 velocity=3.14
- joint wrist3: limit lower=-3.14 upper=3.14 effort=10 velocity=3.14 -> lower=-6.0 upper=6.0 effort=10 velocity=3.14

File: rbpodo_moveit_config/rb5_850e_moveit_config/config/rb5_850e.urdf (robot description, URDF)
Before this commit: robot rb5_850e, 8 links, 7 joints
Joints:
- joint base: limit lower=-3.14 upper=3.14 effort=10 velocity=3.14 -> lower=-6.0 upper=6.0 effort=10 velocity=3.14
- joint shoulder: limit lower=-3.14 upper=3.14 effort=10 velocity=3.14 -> lower=-6.0 upper=6.0 effort=10 velocity=3.14
- joint wrist1: limit lower=-3.14 upper=3.14 effort=10 velocity=3.14 -> lower=-6.0 upper=6.0 effort=10 velocity=3.14
- joint wrist2: limit lower=-3.14 upper=3.14 effort=10 velocity=3.14 -> lower=-6.0 upper=6.0 effort=10 velocity=3.14

Commit message: fix: typo and limit fixed

File: rbpodo_description/robots/rb5_850e.urdf (robot description, URDF)
Before this commit: robot rb5_850e, 8 links, 7 joints
Joints:
- joint base: limit lower=-3.14 upper=3.14 effort=10 velocity=3.14 -> lower=-6.28 upper=6.28 effort=10 velocity=3.14
- joint elbow: limit lower=-3.14 upper=3.14 effort=10 velocity=3.14 -> lower=-6.28 upper=6.28 effort=10 velocity=3.14
- joint shoulder: limit lower=-3.14 upper=3.14 effort=10 velocity=3.14 -> lower=-6.28 upper=6.28 effort=10 velocity=3.14
- joint wrist1: limit lower=-3.14 upper=3.14 effort=10 velocity=3.14 -> lower=-6.28 upper=6.28 effort=10 velocity=3.14
- joint wrist2: limit lower=-3.14 upper=3.14 effort=10 velocity=3.14 -> lower=-6.28 upper=6.28 effort=10 velocity=3.14
- joint wrist3: limit lower=-3.14 upper=3.14 effort=10 velocity=3.14 -> lower=-6.28 upper=6.28 effort=10 velocity=3.14

File: rbpodo_description/robots/rb_6dof.ros2_control.xacro (robot description, xacro)
@@ -23,4 +23,5 @@
           <command_interface name="position"/>
           <state_interface name="position"/>
+          <state_interface name="velocity"/>
           <state_interface name="effort"/>
         </joint>

Commit message: updated joint limit
Signed-off-by: lachan <qhrejddlvltm@gmail.com>

File: rbpodo_description/robots/rb5_850e.urdf (robot description, URDF)
Before this commit: robot rb5_850e, 8 links, 7 joints
Joints:
- joint base: limit lower=-3.14 upper=3.14 effort=10 velocity=3.14 -> lower=-3.14159 upper=3.14159 effort=10 velocity=3.14159
- joint elbow: limit lower=-3.14 upper=3.14 effort=10 velocity=3.14 -> lower=-3.14159 upper=3.14159 effort=10 velocity=3.14159
- joint shoulder: limit lower=-3.14 upper=3.14 effort=10 velocity=3.14 -> lower=-3.14159 upper=3.14159 effort=10 velocity=3.14159
- joint wrist1: limit lower=-3.14 upper=3.14 effort=10 velocity=3.14 -> lower=-3.14159 upper=3.14159 effort=10 velocity=3.14159
- joint wrist2: limit lower=-3.14 upper=3.14 effort=10 velocity=3.14 -> lower=-3.14159 upper=3.14159 effort=10 velocity=3.14159
- joint wrist3: limit lower=-3.14 upper=3.14 effort=10 velocity=3.14 -> lower=-3.14159 upper=3.14159 effort=10 velocity=3.14159
