Commit message: updated prefix configurationg
Signed-off-by: lachan <qhrejddlvltm@gmail.com>

File: rbpodo_description/robots/rb_6dof.xacro (robot description, xacro)
@@ -1,8 +1,8 @@
 <?xml version='1.0' encoding='utf-8'?>
 <robot xmlns:xacro="http://www.ros.org/wiki/xacro">
-  <xacro:macro name="link" params="name model_id:=^ has_inertial:=true">
+  <xacro:macro name="link" params="name prefix:='' model_id:=^ has_inertial:=true">
     <xacro:property name="links_props_file" value="$(find rbpodo_description)/robots/${model_id}/link.yaml" />
     <xacro:property name="links_props" value="${xacro.load_yaml(links_props_file)}" />
-    <link name="${name}">
+    <link name="${prefix}${name}">
       <visual>
         <geometry>
@@ -28,10 +28,10 @@
     </link>
   </xacro:macro>
-  <xacro:macro name="joint" params="name model_id:=^">
+  <xacro:macro name="joint" params="name prefix:='' model_id:=^">
     <xacro:property name="joints_props_file" value="$(find rbpodo_description)/robots/${model_id}/joint.yaml" />
     <xacro:property name="joints_props" value="${xacro.load_yaml(joints_props_file)}" />
     <!-- Check whether name is in joints_props or not -->
     <xacro:property name="props" value="${joints_props[name]}" />
-    <joint name="${name}" type="revolute">
+    <joint name="${prefix}${name}" type="revolute">
       <origin xyz="${props.origin.xyz}" rpy="${props.origin.rpy}" />
       <parent link="${props.parent}" />
@@ -43,18 +43,18 @@
   </xacro:macro>
   <xacro:macro name="rb_6dof" params="model_id prefix='' tcp_name='tcp' tcp_xyz='0 0 0' tcp_rpy='0 0 0'">
-    <xacro:link name="${prefix}link0" has_inertial="false" />
-    <xacro:link name="${prefix}link1" />
-    <xacro:link name="${prefix}link2" />
-    <xacro:link name="${prefix}link3" />
-    <xacro:link name="${prefix}link4" />
-    <xacro:link name="${prefix}link5" />
-    <xacro:link name="${prefix}link6" />
+    <xacro:link name="link0" prefix="${prefix}" has_inertial="false" />
+    <xacro:link name="link1" prefix="${prefix}" />
+    <xacro:link name="link2" prefix="${prefix}" />
+    <xacro:link name="link3" prefix="${prefix}" />
+    <xacro:link name="link4" prefix="${prefix}" />
+    <xacro:link name="link5" prefix="${prefix}" />
+    <xacro:link name="link6" prefix="${prefix}" />
     <link name="${prefix}${tcp_name}" />
-    <xacro:joint name="${prefix}base" />
-    <xacro:joint name="${prefix}shoulder" />
-    <xacro:joint name="${prefix}elbow" />
-    <xacro:joint name="${prefix}wrist1" />
-    <xacro:joint name="${prefix}wrist2" />
-    <xacro:joint name="${prefix}wrist3" />
+    <xacro:joint name="base"      prefix="${prefix}"/>
+    <xacro:joint name="shoulder"  prefix="${prefix}"/>
+    <xacro:joint name="elbow"     prefix="${prefix}"/>
+    <xacro:joint name="wrist1"    prefix="${prefix}"/>
+    <xacro:joint name="wrist2"    prefix="${prefix}"/>
+    <xacro:joint name="wrist3"    prefix="${prefix}"/>
     <joint name="${prefix}${tcp_name}_joint" type="fixed">
       <origin xyz="${tcp_xyz}" rpy="${tcp_rpy}" />

Commit message: fix joint macro
Signed-off-by: lachan <qhrejddlvltm@gmail.com>

File: rbpodo_description/robots/rb_6dof.xacro (robot description, xacro)
@@ -35,6 +35,6 @@
     <joint name="${prefix}${name}" type="revolute">
       <origin xyz="${props.origin.xyz}" rpy="${props.origin.rpy}" />
-      <parent link="${props.parent}" />
-      <child link="${props.child}" />
+      <parent link="${prefix}${props.parent}" />
+      <child link="${prefix}${props.child}" />
       <axis xyz="${props.axis.xyz}" />
       <xacro:property name="limit" value="${props.limit}" />
@@ -44,5 +44,5 @@
   <xacro:macro name="rb_6dof" params="model_id prefix='' tcp_name='tcp' tcp_xyz='0 0 0' tcp_rpy='0 0 0'">
     <xacro:link name="link0" prefix="${prefix}" has_inertial="false" />
-    <xacro:link name="link1" prefix="${prefix}" />
+    <xacro:link name="link1" s="${prefix}" />
     <xacro:link name="link2" prefix="${prefix}" />
     <xacro:link name="link3" prefix="${prefix}" />
